Commit message: update

File: robot_model/description/robot_core.xacro (robot description, xacro)
@@ -34,11 +34,23 @@
     <link name="chassis">
         <visual>
-            <origin xyz="0.25 0.0 0.075" rpy="0.0 0.0 0.0" />
+            <origin xyz="0.25 0 0.075"/>
             <geometry>
-                <box size="0.5 0.3 0.12" />
+                <box size="0.5 0.3 0.12"/>
             </geometry>
-            <material name="white" />
+            <material name="white"/>
         </visual>
+        <collision>
+            <origin xyz="0.25 0 0.075"/>
+            <geometry>
+                <box size="0.5 0.3 0.12"/>
+            </geometry>
+        </collision>
+        <xacro:inertial_box mass="0.5" x="0.3" y="0.3" z="0.15">
+            <origin xyz="0.15 0 0.075" rpy="0 0 0"/>
+        </xacro:inertial_box>
     </link>
+    <gazebo reference="chassis">
+        <material>Gazebo/White</material>
+    </gazebo>
       <!-- LEFT WHEEL 2 LINK -->
       <joint name="left_wheel_joint_2" type="continuous">
@@ -60,8 +72,11 @@
             </geometry>
         </collision>
-        <xacro:inertial_cylinder mass="0.1" length="0.04" radius="0.05">
+        <xacro:inertial_cylinder mass="0.1" length="0.045" radius="0.05">
             <origin xyz="0 0 0" rpy="0 0 0"/>
         </xacro:inertial_cylinder>
     </link>
+    <gazebo reference="left_wheel_2">
+        <material>Gazebo/Blue</material>
+    </gazebo>
     <!-- LEFT WHEEL 1 LINK -->
     <joint name="left_wheel_joint_1" type="continuous">
@@ -83,8 +98,11 @@
             </geometry>
         </collision>
-        <xacro:inertial_cylinder mass="0.1" length="0.04" radius="0.05">
+        <xacro:inertial_cylinder mass="0.1" length="0.045" radius="0.05">
             <origin xyz="0 0 0" rpy="0 0 0"/>
         </xacro:inertial_cylinder>
     </link>
+    <gazebo reference="left_wheel_1">
+        <material>Gazebo/Blue</material>
+    </gazebo>
     <!-- RIGHT WHEEL 2 LINK -->
     <joint name="right_wheel_joint_2" type="continuous">
@@ -106,8 +124,11 @@
             </geometry>
         </collision>
-        <xacro:inertial_cylinder mass="0.1" length="0.04" radius="0.05">
+        <xacro:inertial_cylinder mass="0.1" length="0.045" radius="0.05">
             <origin xyz="0 0 0" rpy="0 0 0"/>
         </xacro:inertial_cylinder>
     </link>
+    <gazebo reference="right_wheel_2">
+        <material>Gazebo/Blue</material>
+    </gazebo>
       <!-- RIGHT WHEEL 1 LINK -->
       <joint name="right_wheel_joint_1" type="continuous">
@@ -129,7 +150,10 @@
             </geometry>
         </collision>
-        <xacro:inertial_cylinder mass="0.1" length="0.04" radius="0.05">
+        <xacro:inertial_cylinder mass="0.1" length="0.045" radius="0.05">
             <origin xyz="0 0 0" rpy="0 0 0"/>
         </xacro:inertial_cylinder>
     </link>
+    <gazebo reference="right_wheel_1">
+        <material>Gazebo/Blue</material>
+    </gazebo>
 </robot>

Commit message: update file joint state

File: robot_model/description/robot_core.xacro (robot description, xacro)
@@ -50,7 +50,4 @@
         </xacro:inertial_box>
     </link>
-    <gazebo reference="chassis">
-        <material>Gazebo/White</material>
-    </gazebo>
       <!-- LEFT WHEEL 2 LINK -->
       <joint name="left_wheel_joint_2" type="continuous">
@@ -76,7 +73,4 @@
         </xacro:inertial_cylinder>
     </link>
-    <gazebo reference="left_wheel_2">
-        <material>Gazebo/Blue</material>
-    </gazebo>
     <!-- LEFT WHEEL 1 LINK -->
     <joint name="left_wheel_joint_1" type="continuous">
@@ -102,7 +96,4 @@
         </xacro:inertial_cylinder>
     </link>
-    <gazebo reference="left_wheel_1">
-        <material>Gazebo/Blue</material>
-    </gazebo>
     <!-- RIGHT WHEEL 2 LINK -->
     <joint name="right_wheel_joint_2" type="continuous">
@@ -128,7 +119,4 @@
         </xacro:inertial_cylinder>
     </link>
-    <gazebo reference="right_wheel_2">
-        <material>Gazebo/Blue</material>
-    </gazebo>
       <!-- RIGHT WHEEL 1 LINK -->
       <joint name="right_wheel_joint_1" type="continuous">
@@ -154,6 +142,3 @@
         </xacro:inertial_cylinder>
     </link>
-    <gazebo reference="right_wheel_1">
-        <material>Gazebo/Blue</material>
-    </gazebo>
 </robot>

Commit message: update file

File: robot_model/description/robot_core.xacro (robot description, xacro)
@@ -100,6 +100,6 @@
         <parent link="base_link" />
         <child link="right_wheel_2" />
-        <origin xyz="-0.125 -0.175 0" rpy="${pi/2} 0 0" />
-        <axis xyz="0 0 -1"/>
+        <origin xyz="-0.125 -0.175 0" rpy="${-pi/2} 0 0" />
+        <axis xyz="0 0 1"/>
     </joint>
     <link name="right_wheel_2">
@@ -123,6 +123,6 @@
         <parent link="base_link" />
         <child link="right_wheel_1" />
-        <origin xyz="0.125 -0.175 0" rpy="${pi/2} 0 0" />
-        <axis xyz="0 0 -1"/>
+        <origin xyz="0.125 -0.175 0" rpy="${-pi/2} 0 0" />
+        <axis xyz="0 0 1"/>
     </joint>
     <link name="right_wheel_1">
