Commit message: update slam

File: robot_model/description/lidar.xacro (robot description, xacro)
@@ -2,5 +2,5 @@
 <robot xmlns:xacro="http://www.ros.org/wiki/xacro" >
     <joint name="lidar_joint" type="fixed">
-        <parent link="chassis"/>
+        <parent link="base_link"/>
         <child link="lidar_link"/>
         <origin xyz="0.45 0.0 0.16" rpy="0 0 0"/>

Commit message: update nav2

File: robot_model/description/lidar.xacro (robot description, xacro)
@@ -2,5 +2,5 @@
 <robot xmlns:xacro="http://www.ros.org/wiki/xacro" >
     <joint name="lidar_joint" type="fixed">
-        <parent link="base_link"/>
+        <parent link="chassis"/>
         <child link="lidar_link"/>
         <origin xyz="0.45 0.0 0.16" rpy="0 0 0"/>
